File: hardware/atm128_kicad/atm128.kicad_pcb (KiCad board)
At the start: 2 copper layers, 76.2 x 55.9 mm, 54 parts, among them J1 Power Jack, J2 Conn_02x16_Odd_Even, J3 Conn_02x16_Odd_Even, J4 ISP, J5 JTAG, J6 USB_C_Receptacle_USB2.0, U1 LM2596S-5, U2 ATmega128-16A, U4 CH340E

Commit message: feat: add TNOW LED, complete review for rev1.0
Parts:
- added D8: TNOW, LED_SMD:LED_0805_2012Metric, F.Cu at (83.4, 61.3)
- added R11: 1k, Resistor_SMD:R_0805_2012Metric, F.Cu at (83.4, 63.3)
Connections:
- U4 pad 6: unconnected-(U4-Pad6) -> /tnow
Routing:
- net +5V: track 340.2 -> 323.9 mm
- net /power_in: track 31.2 -> 19.2 mm
- net /tnow: track 0.00 -> 7.91 mm, vias 0 -> 2
- net Net-(D8-Pad2): track 0.00 -> 2.05 mm
- net /nRST: track 118.4 -> 117.5 mm
- net /TXD0: track 22.1 -> 21.5 mm
- net GND: track 85.3 -> 84.9 mm, vias 139 -> 161
